Commit message: tried new robot

File: Tutorial-1-Intro/template_mujoco_python/horton_urdf_files.urdf (robot description, URDF)
Before this commit: robot horton_urdf_files, 4 links, 3 joints
Links:
- link l_foot: geometry collision mesh filename=l_foot.STL; visual mesh filename=l_foot.STL
- link l_leg: geometry collision mesh filename=l_leg.STL; visual mesh filename=l_leg.STL
- link r_foot: geometry collision mesh filename=r_foot.STL; visual mesh filename=r_foot.STL
- link r_leg: geometry collision mesh filename=r_leg.STL; visual mesh filename=r_leg.STL
