Commit message: added converted mjcf and it kinda works

File: my-robot-fixed/robot.urdf (robot description, URDF)
Before this commit: robot onshape, 2 links, 1 joints
Links:
- added link left_leg_1, mass 1e-9; collision mesh filename=right_arm.stl; visual mesh filename=right_arm.stl
- added link left_leg_2, mass 1e-9; collision mesh filename=right_battery.stl; visual mesh filename=right_battery.stl
- added link left_leg_3, mass 1e-9; collision mesh filename=left_foot.stl; visual mesh filename=left_foot.stl
- added link left_leg_4, mass 1e-9; collision mesh filename=left_leg.stl; visual mesh filename=left_leg.stl
- added link right_leg_1, mass 1e-9; collision mesh filename=left_arm.stl; visual mesh filename=left_arm.stl
- added link right_leg_2; collision mesh filename=right_foot.stl; visual mesh filename=right_foot.stl
- added link right_leg_3, mass 1e-9; collision mesh filename=right_leg.stl; visual mesh filename=right_leg.stl
- added link right_leg_4, mass 1e-9; collision mesh filename=right_battery.stl; visual mesh filename=right_battery.stl
- link left_leg: geometry 
- link right_leg: geometry 
Joints:
- added joint left_leg_1_fixing: type fixed, parent left_leg, child left_leg_1, origin xyz=0 0 0 rpy=0 -0 0, axis 0 0 1, limit effort=1 velocity=20
- added joint left_leg_2_fixing: type fixed, parent left_leg, child left_leg_2, origin xyz=0 0 0 rpy=0 -0 0, axis 0 0 1, limit effort=1 velocity=20
- added joint left_leg_3_fixing: type fixed, parent left_leg, child left_leg_3, origin xyz=0 0 0 rpy=0 -0 0, axis 0 0 1, limit effort=1 velocity=20
- added joint left_leg_4_fixing: type fixed, parent left_leg, child left_leg_4, origin xyz=0 0 0 rpy=0 -0 0, axis 0 0 1, limit effort=1 velocity=20
- added joint right_leg_1_fixing: type fixed, parent right_leg, child right_leg_1, origin xyz=0 0 0 rpy=0 -0 0, axis 0 0 1, limit effort=1 velocity=20
- added joint right_leg_2_fixing: type fixed, parent right_leg, child right_leg_2, origin xyz=0 0 0 rpy=0 -0 0, axis 0 0 1, limit effort=1 velocity=20
- added joint right_leg_3_fixing: type fixed, parent right_leg, child right_leg_3, origin xyz=0 0 0 rpy=0 -0 0, axis 0 0 1, limit effort=1 velocity=20
- added joint right_leg_4_fixing: type fixed, parent right_leg, child right_leg_4, origin xyz=0 0 0 rpy=0 -0 0, axis 0 0 1, limit effort=1 velocity=20
